File: tests/golden/ecc83_srpp.pour_gnd.seed42.kicad_pcb (KiCad board)
At the start: 2 copper layers, 52 x 46 mm, 15 parts, among them J1 J_HTR, J2 J_IN, J3 J_OUT, J4 J_PWR, U2 u1_V

Commit message: synthesizer: no more duplicate same-named nets — chain-opening pins reuse their net
- root cause: two connection chains opening on the SAME pin
  (`r_top.2 -> r_bot…; r_top.2 -> r_m1…`) each minted a fresh auto_*
  net with the same name — one solver node (converter coalesces by
  name), two NetIds for anyone keying by id (the fault campaign's
  original short-merge silently missed the copy)
- fix at both creation sites in hierarchical_connectivity: a chain
  opening on an already-connected pin REUSES the pin's existing net
- regression test: net-name uniqueness asserted on three fixtures (the
  fault-campaign one previously carried the dupe)
- ecc83 golden re-blessed: the change is a pure net RENAME (first
  creation's name now wins) — proven 17/17 pad→net-number assignments
  identical, all 15,016 geometry lines byte-identical, net counts equal;
  guard green again
- safety fixtures opt out of the layout sweep via a `bhdl-sweep: skip`
  marker (user decision: safety-engine fixtures are not layout targets
  and must not pollute the parked layout baseline)
- fault_campaign's by-name merge stays as defense in depth

Co-Authored-By: Claude Fable 5 <noreply@anthropic.com>
Connections:
- net auto_J_OUT_1 renamed auto_c_out_2
- net auto_u1_G1 renamed auto_J_IN_1
- net auto_u1_G2 renamed auto_u1_A1
- net auto_u1_K2 renamed auto_r_kup_2
Changed lines of the file:
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@@
   (net 2 "HTR")
   (net 3 "VBB")
-  (net 4 "auto_u1_G1")
+  (net 4 "auto_J_IN_1")
   (net 5 "auto_u1_K1")
-  (net 6 "auto_u1_G2")
-  (net 7 "auto_u1_K2")
-  (net 8 "auto_J_OUT_1")
+  (net 6 "auto_u1_A1")
+  (net 7 "auto_r_kup_2")
+  (net 8 "auto_c_out_2")
   (gr_rect (start 0 0) (end 52 46) (layer "Edge.Cuts") (stroke (width 0.05) (type solid)) (fill none))
   (footprint "MountingHole_3.2mm" (layer "F.Cu") (at 3.8 3.8)
@@
     (property "Reference" "J2" (at 3.450 -0.000 0) (layer "F.SilkS") (effects (font (size 1 1) (thickness 0.150))))
     (property "Value" "J_IN" (at 0 6 0) (layer "F.Fab") (effects (font (size 1 1) (thickness 0.15))))
-    (pad "1" thru_hole rect (at 0 -2.5 270.0) (size 3 3) (drill 1.5) (layers "*.Cu" "*.Mask") (net 4 "auto_u1_G1"))
+    (pad "1" thru_hole rect (at 0 -2.5 270.0) (size 3 3) (drill 1.5) (layers "*.Cu" "*.Mask") (net 4 "auto_J_IN_1"))
     (pad "2" thru_hole oval (at 0 2.5 270.0) (size 3 3) (drill 1.5) (layers "*.Cu" "*.Mask") (net 1 "GND"))
   )
@@
     (property "Reference" "J3" (at -3.450 0.000 0) (layer "F.SilkS") (effects (font (size 1 1) (thickness 0.150))))
     (property "Value" "J_OUT" (at 0 6 0) (layer "F.Fab") (effects (font (size 1 1) (thickness 0.15))))
-    (pad "1" thru_hole rect (at 0 -2.5 90.0) (size 3 3) (drill 1.5) (layers "*.Cu" "*.Mask") (net 8 "auto_J_OUT_1"))
+    (pad "1" thru_hole rect (at 0 -2.5 90.0) (size 3 3) (drill 1.5) (layers "*.Cu" "*.Mask") (net 8 "auto_c_out_2"))
     (pad "2" thru_hole oval (at 0 2.5 90.0) (size 3 3) (drill 1.5) (layers "*.Cu" "*.Mask") (net 1 "GND"))
   )
@@
     (property "Reference" "R3" (at 0.000 2.700 0) (layer "F.SilkS") (effects (font (size 1 1) (thickness 0.150))))
     (property "Value" "r_leak" (at 0 2.25 0) (layer "F.Fab") (effects (font (size 1 1) (thickness 0.15))))
-    (pad "1" thru_hole rect (at -3.81 0 90.0) (size 1.6 1.6) (drill 0.8) (layers "*.Cu" "*.Mask") (net 4 "auto_u1_G1"))
+    (pad "1" thru_hole rect (at -3.81 0 90.0) (size 1.6 1.6) (drill 0.8) (layers "*.Cu" "*.Mask") (net 4 "auto_J_IN_1"))
     (pad "2" thru_hole oval (at 3.81 0 90.0) (size 1.6 1.6) (drill 0.8) (layers "*.Cu" "*.Mask") (net 1 "GND"))
   )
@@
     (property "Reference" "R2" (at -5.560 0.000 0) (layer "F.SilkS") (effects (font (size 1 1) (thickness 0.150))))
     (property "Value" "r_kup" (at 0 2.25 0) (layer "F.Fab") (effects (font (size 1 1) (thickness 0.15))))
-    (pad "1" thru_hole rect (at -3.81 0 90.0) (size 1.6 1.6) (drill 0.8) (layers "*.Cu" "*.Mask") (net 6 "auto_u1_G2"))
-    (pad "2" thru_hole oval (at 3.81 0 90.0) (size 1.6 1.6) (drill 0.8) (layers "*.Cu" "*.Mask") (net 7 "auto_u1_K2"))
+    (pad "1" thru_hole rect (at -3.81 0 90.0) (size 1.6 1.6) (drill 0.8) (layers "*.Cu" "*.Mask") (net 6 "auto_u1_A1"))
+    (pad "2" thru_hole oval (at 3.81 0 90.0) (size 1.6 1.6) (drill 0.8) (layers "*.Cu" "*.Mask") (net 7 "auto_r_kup_2"))
   )
   (footprint "Disc-P5.00" (layer "F.Cu") (at 15.9 34.9 270.0)
     (property "Reference" "C1" (at 4.250 -0.000 0) (layer "F.SilkS") (effects (font (size 1 1) (thickness 0.150))))
     (property "Value" "c_out" (at 0 2.25 0) (layer "F.Fab") (effects (font (size 1 1) (thickness 0.15))))
-    (pad "1" thru_hole rect (at -2.5 0 270.0) (size 1.6 1.6) (drill 0.8) (layers "*.Cu" "*.Mask") (net 7 "auto_u1_K2"))
-    (pad "2" thru_hole oval (at 2.5 0 270.0) (size 1.6 1.6) (drill 0.8) (layers "*.Cu" "*.Mask") (net 8 "auto_J_OUT_1"))
+    (pad "1" thru_hole rect (at -2.5 0 270.0) (size 1.6 1.6) (drill 0.8) (layers "*.Cu" "*.Mask") (net 7 "auto_r_kup_2"))
+    (pad "2" thru_hole oval (at 2.5 0 270.0) (size 1.6 1.6) (drill 0.8) (layers "*.Cu" "*.Mask") (net 8 "auto_c_out_2"))
   )
   (footprint "Axial-P7.62" (layer "F.Cu") (at 12.7 34.9 180.0)
     (property "Reference" "R4" (at -6.060 0.000 0) (layer "F.SilkS") (effects (font (size 1 1) (thickness 0.150))))
     (property "Value" "r_load" (at 0 2.25 0) (layer "F.Fab") (effects (font (size 1 1) (thickness 0.15))))
-    (pad "1" thru_hole rect (at -3.81 0 180.0) (size 1.6 1.6) (drill 0.8) (layers "*.Cu" "*.Mask") (net 8 "auto_J_OUT_1"))
+    (pad "1" thru_hole rect (at -3.81 0 180.0) (size 1.6 1.6) (drill 0.8) (layers "*.Cu" "*.Mask") (net 8 "auto_c_out_2"))
     (pad "2" thru_hole oval (at 3.81 0 180.0) (size 1.6 1.6) (drill 0.8) (layers "*.Cu" "*.Mask") (net 1 "GND"))
   )
@@
     (property "Reference" "U2" (at 8.100 -0.113 0) (layer "F.SilkS") (effects (font (size 1 1) (thickness 0.150))))
     (property "Value" "u1_V" (at 0 7.762500000000001 0) (layer "F.Fab") (effects (font (size 1 1) (thickness 0.15))))
-    (pad "1" thru_hole rect (at 3.45 4.8 -0.0) (size 2.0500000000000003 2.0500000000000003) (drill 1.02) (layers "*.Cu" "*.Mask") (net 6 "auto_u1_G2"))
-    (pad "2" thru_hole oval (at 5.6000000000000005 1.87 -0.0) (size 2.0500000000000003 2.0500000000000003) (drill 1.02) (layers "*.Cu" "*.Mask") (net 4 "auto_u1_G1"))
+    (pad "1" thru_hole rect (at 3.45 4.8 -0.0) (size 2.0500000000000003 2.0500000000000003) (drill 1.02) (layers "*.Cu" "*.Mask") (net 6 "auto_u1_A1"))
+    (pad "2" thru_hole oval (at 5.6000000000000005 1.87 -0.0) (size 2.0500000000000003 2.0500000000000003) (drill 1.02) (layers "*.Cu" "*.Mask") (net 4 "auto_J_IN_1"))
     (pad "3" thru_hole oval (at 5.6000000000000005 -1.78 -0.0) (size 2.0500000000000003 2.0500000000000003) (drill 1.02) (layers "*.Cu" "*.Mask") (net 5 "auto_u1_K1"))
     (pad "4" thru_hole oval (at 3.45 -4.71 -0.0) (size 2.0500000000000003 2.0500000000000003) (drill 1.02) (layers "*.Cu" "*.Mask") (net 2 "HTR"))
     (pad "5" thru_hole oval (at 0 -5.8500000000000005 -0.0) (size 2.0500000000000003 2.0500000000000003) (drill 1.02) (layers "*.Cu" "*.Mask") (net 2 "HTR"))
     (pad "6" thru_hole oval (at -3.46 -4.71 -0.0) (size 2.0500000000000003 2.0500000000000003) (drill 1.02) (layers "*.Cu" "*.Mask") (net 3 "VBB"))
-    (pad "7" thru_hole oval (at -5.61 -1.78 -0.0) (size 2.0500000000000003 2.0500000000000003) (drill 1.02) (layers "*.Cu" "*.Mask") (net 6 "auto_u1_G2"))
-    (pad "8" thru_hole oval (at -5.61 1.83 -0.0) (size 2.0500000000000003 2.0500000000000003) (drill 1.02) (layers "*.Cu" "*.Mask") (net 7 "auto_u1_K2"))
+    (pad "7" thru_hole oval (at -5.61 -1.78 -0.0) (size 2.0500000000000003 2.0500000000000003) (drill 1.02) (layers "*.Cu" "*.Mask") (net 6 "auto_u1_A1"))
+    (pad "8" thru_hole oval (at -5.61 1.83 -0.0) (size 2.0500000000000003 2.0500000000000003) (drill 1.02) (layers "*.Cu" "*.Mask") (net 7 "auto_r_kup_2"))
     (pad "9" thru_hole oval (at -3.46 4.8 -0.0) (size 2.0500000000000003 2.0500000000000003) (drill 1.02) (layers "*.Cu" "*.Mask") (net 1 "GND"))
   )
